File: OpenC64MegaDrivePadAdapter.kicad_pcb (KiCad board)
At the start: 2 copper layers, 52.9 x 31 mm, 17 parts, among them J10 DB9_F_TO_C64, J20 DB9_M_TO_PAD, Q1 BC547

Commit message: V4 PCB
Routing:
- net GND: track 101.8 -> 154.2 mm
Changed lines of the file:
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@@
     (thickness 1.6)
     (drawings 140)
-    (tracks 197)
+    (tracks 207)
     (zones 0)
     (modules 17)
@@
   (via (at 155.646534 113.565448) (size 1) (drill 0.8) (layers F.Cu B.Cu) (net 15))
   (segment (start 180.424 102.452) (end 180.424 101.704) (width 0.1) (layer F.Cu) (net 15))
-  (segment (start 180.424 101.704) (end 179.12 100.4) (width 0.1) (layer F.Cu) (net 15))
-  (segment (start 181.53 96.61) (end 184.488 96.61) (width 0.1) (layer F.Cu) (net 15))
-  (segment (start 179.12 100.4) (end 179.12 99.02) (width 0.1) (layer F.Cu) (net 15))
-  (segment (start 179.12 99.02) (end 181.53 96.61) (width 0.1) (layer F.Cu) (net 15))
   (segment (start 142.654 102.45344) (end 140.20544 102.45344) (width 0.5) (layer F.Cu) (net 15))
   (segment (start 140.20544 102.45344) (end 139.352 101.6) (width 0.5) (layer F.Cu) (net 15))
@@
   (segment (start 139.352 116.84) (end 143.416 116.84) (width 0.1) (layer F.Cu) (net 15))
   (segment (start 155.646534 116.065448) (end 155.646534 113.565448) (width 0.1) (layer B.Cu) (net 15))
+  (segment (start 184.488 94.07) (end 184.314 94.07) (width 0.25) (layer F.Cu) (net 15))
+  (segment (start 184.314 94.07) (end 183.388 94.996) (width 0.25) (layer F.Cu) (net 15))
+  (segment (start 183.388 94.996) (end 176.022 94.996) (width 0.25) (layer F.Cu) (net 15))
+  (segment (start 176.86656 118.618) (end 179.154 116.33056) (width 0.1) (layer F.Cu) (net 15))
+  (segment (start 146.05 118.618) (end 176.86656 118.618) (width 0.1) (layer F.Cu) (net 15))
+  (segment (start 143.924 116.492) (end 146.05 118.618) (width 0.1) (layer F.Cu) (net 15))
+  (segment (start 143.924 116.332) (end 143.924 116.492) (width 0.1) (layer F.Cu) (net 15))
+  (segment (start 180.758 96.61) (end 184.488 96.61) (width 0.25) (layer F.Cu) (net 15))
+  (segment (start 180.424 102.452) (end 180.424 101.684) (width 0.25) (layer F.Cu) (net 15))
+  (segment (start 180.424 101.684) (end 179.07 100.33) (width 0.25) (layer F.Cu) (net 15))
+  (segment (start 179.07 100.33) (end 179.07 98.298) (width 0.25) (layer F.Cu) (net 15))
+  (segment (start 179.07 98.298) (end 180.758 96.61) (width 0.25) (layer F.Cu) (net 15))
+  (segment (start 173.676 92.65) (end 176.022 94.996) (width 0.25) (layer F.Cu) (net 15))
+  (segment (start 171.94 92.65) (end 173.676 92.65) (width 0.25) (layer F.Cu) (net 15))
   (segment (start 169.4 94.506) (end 169.4 92.65) (width 0.25) (layer B.Cu) (net 16))
   (segment (start 168.352 95.554) (end 169.4 94.506) (width 0.25) (layer B.Cu) (net 16))

Commit message: Minor changes
Parts:
- removed G***: LOGO, oshw:LOGO
- removed G***: LOGO, mdpad:LOGO
- added V1: PAD_LOGO, OpenC64MegaDrivePadAdapter:LOGO, F.Cu at (151.9, 96.8)
- added V2: OSHW, OpenC64MegaDrivePadAdapter:oshw, B.Cu at (151.8, 100.5)
Connections:
- J10 pad : GND -> (no net)
- J20 pad : GND -> (no net)
Routing:
- net GND: track 154.2 -> 101.2 mm

Commit message: rev. 5 PCB
Parts:
- added Q2: BC547, TO_SOT_Packages_THT:TO-92_Molded_Narrow, F.Cu at (168.4, 93.8)
- added R1: 10k, Resistors_THT:R_Axial_DIN0204_L3.6mm_D1.6mm_P7.62mm_Horizontal, F.Cu at (166.7, 105.1)
- R2: value 2.2k -> 10k
- R4: value 100k -> 10k
- moved R4 7.38 mm to (174.3, 96.9), turned to 180 degrees
- moved R2 6.19 mm to (174.3, 102.4), turned to 180 degrees
- moved S2 6.05 mm to (171.0, 111.3), turned to 270 degrees
- moved S1 5.90 mm to (163.2, 111.3), turned to 270 degrees
- moved S3 5.90 mm to (152.5, 111.3), turned to 270 degrees
- moved R3 5.80 mm to (174.3, 99.6), turned to 180 degrees
- moved Q1 3.42 mm to (172.5, 91.2), turned to 270 degrees
- moved D6 1.44 mm to (164.1, 105.1)
- moved D5 1.31 mm to (164.2, 102.4)
- moved D4 1.17 mm to (164.2, 99.6)
- moved D3 1.05 mm to (164.2, 96.9)
- moved D2 0.96 mm to (164.2, 94.1)
- moved D1 0.92 mm to (164.2, 91.4)
- moved V2 0.70 mm to (151.1, 100.5)
- moved V1 0.38 mm to (151.5, 96.8)
Connections:
- J10 pad : (no net) -> GND
- J20 pad : (no net) -> GND
- R2 pad 2: Net-(Q1-Pad1) -> Net-(R1-Pad1)
- R3 pad 1: Net-(R3-Pad1) -> +5V
- R3 pad 2: +5V -> Net-(Q1-Pad1)
- R4 pad 1: Net-(R3-Pad1) -> +5V
- R4 pad 2: Net-(Q1-Pad2) -> Net-(Q2-Pad1)
- S1 pad 2: /md_c/~st -> /md_b/~a
- S1 pad 5: /md_b/~a -> /md_c/~st
- S2 pad 1: Net-(R3-Pad1) -> Net-(S2-Pad1)
- S2 pad 2: Net-(S1-Pad3) -> Net-(S2-Pad2)
- S2 pad 3: Net-(D5-Pad1) -> Net-(S2-Pad3)
- S2 pad 4: Net-(S2-Pad4) -> Net-(D5-Pad1)
- S2 pad 5: Net-(S2-Pad5) -> Net-(S1-Pad3)
- S2 pad 6: Net-(S2-Pad6) -> Net-(R1-Pad1)
- S3 pad 1: Net-(R3-Pad1) -> GND
- S3 pad 2: /pot_x -> Net-(Q2-Pad2)
- S3 pad 4: Net-(S3-Pad4) -> Net-(Q1-Pad1)
- S3 pad 5: Net-(S3-Pad5) -> /pot_x
- S3 pad 6: Net-(S3-Pad6) -> Net-(Q2-Pad1)
Routing:
- net GND: track 101.2 -> 54.4 mm
- net Net-(Q2-Pad1): track 0.00 -> 42.0 mm
- net Net-(R3-Pad1): track 35.2 -> 0.00 mm
- net Net-(Q2-Pad2): track 0.00 -> 29.9 mm
- net Net-(R1-Pad1): track 0.00 -> 16.0 mm
- net Net-(Q1-Pad1): track 43.9 -> 58.8 mm
- net Net-(D4-Pad1): track 29.1 -> 19.9 mm
- net Net-(Q1-Pad2): track 6.05 -> 13.7 mm
- net /md_c/~st: track 40.5 -> 44.3 mm
- net /md_right: track 18.8 -> 21.4 mm
- net /left: track 17.6 -> 15.4 mm
- net Net-(D5-Pad1): track 14.2 -> 12.1 mm
- net /md_up: track 18.5 -> 16.6 mm
- net /md_left: track 19.3 -> 17.7 mm
- net /md_down: track 19.1 -> 17.7 mm
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Other:
- board text added: "rev: 5"
- board text removed: "V4"

Commit message: rev 6
Parts:
- added R5: 10k, Resistor_THT:R_Axial_DIN0204_L3.6mm_D1.6mm_P7.62mm_Horizontal, F.Cu at (174.3, 95.9)
- D1, D2, D3, D4, D5, D6: footprint Diodes_THT:D_DO-35_SOD27_P7.62mm_Horizontal -> Diode_THT:D_DO-35_SOD27_P7.62mm_Horizontal
- J10: footprint db9:DB_9F -> OpenC64MegaDrivePadAdapter:DB_9F
- J20: footprint w_conn_d-sub:DB_9M -> OpenC64MegaDrivePadAdapter:DB_9M
- Q1, Q2: footprint TO_SOT_Packages_THT:TO-92_Molded_Narrow -> Package_TO_SOT_THT:TO-92L_HandSolder
- R1, R2, R3, R4: footprint Resistors_THT:R_Axial_DIN0204_L3.6mm_D1.6mm_P7.62mm_Horizontal -> Resistor_THT:R_Axial_DIN0204_L3.6mm_D1.6mm_P7.62mm_Horizontal
- S1, S2, S3: footprint Buttons_Switches_THT:SW_CuK_JS202011CQN_DPDT_Straight -> Button_Switch_THT:SW_CuK_JS202011CQN_DPDT_Straight
- moved R4 1.35 mm to (174.3, 98.2)
- moved R3 0.90 mm to (174.3, 100.5)
- moved Q1 0.50 mm to (172.5, 90.7)
- moved Q2 0.50 mm to (168.4, 93.3)
- moved R2 0.45 mm to (174.3, 102.8)
Connections:
- J10 pad 5: /pot_y -> /md_sel
- J20 pad 7: +5V -> /md_sel
Routing:
- net /md_sel: track 0.00 -> 42.5 mm
- net +5V: track 62.5 -> 70.2 mm
- net /md_b/~a: track 19.7 -> 23.6 mm
- net Net-(Q1-Pad1): track 58.8 -> 61.1 mm
- net /md_down: track 17.7 -> 19.6 mm
- net /md_right: track 21.4 -> 22.8 mm
- net Net-(Q2-Pad1): track 42.0 -> 40.9 mm
- net /md_left: track 17.7 -> 18.7 mm
Other:
- board text added: "rev: 6"
- board text removed: "rev: 5"
